Commit message: tesseract planner

File: simulation/tes_planner/urdf/combined.urdf (robot description, URDF)
Before this commit: robot combined, 26 links, 25 joints
Joints:
- joint obstacle_joint: origin xyz=0.5 0.0 1.2 rpy=0 0 0 -> xyz=0.8 0.0 1.2 rpy=0 0 0

Commit message: tes_ur_plan

File: simulation/tes_planner/urdf/combined.urdf (robot description, URDF)
Before this commit: robot combined, 26 links, 25 joints
Links:
- removed link obstacle
- added link UR_base_link, mass 4; collision mesh filename=/home/iamnotedible/RR_Project/simulation/models/ur/meshes/u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 scale=1 1 1; visual mesh filename=/home/iamnotedible/RR_Project/simulation/models/ur/meshes/u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 scale=1 1 1
- added link forearm_link, mass 2.275; collision mesh filename=/home/iamnotedible/RR_Project/simulation/models/ur/meshes/u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 scale=1 1 1; visual mesh filename=/home/iamnotedible/RR_Project/simulation/models/ur/meshes/u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 scale=1 1 1
- added link shoulder_link, mass 3.7; collision mesh filename=/home/iamnotedible/RR_Project/simulation/models/ur/meshes/u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 scale=1 1 1; visual mesh filename=/home/iamnotedible/RR_Project/simulation/models/ur/meshes/u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 scale=1 1 1
- added link upper_arm_link, mass 8.393; collision mesh filename=/home/iamnotedible/RR_Project/simulation/models/ur/meshes/u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 scale=1 1 1; visual mesh filename=/home/iamnotedible/RR_Project/simulation/models/ur/meshes/u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 scale=1 1 1
- added link ur_pedestal, mass 1; visual cylinder length=1 radius=0.15
- added link wrist_1_link, mass 1.219; collision mesh filename=/home/iamnotedible/RR_Project/simulation/models/ur/meshes/u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 scale=1 1 1; visual mesh filename=/home/iamnotedible/RR_Project/simulation/models/ur/meshes/u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 scale=1 1 1
- added link wrist_2_link, mass 1.219; collision mesh filename=/home/iamnotedible/RR_Project/simulation/models/ur/meshes/u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 scale=1 1 1; visual mesh filename=/home/iamnotedible/RR_Project/simulation/models/ur/meshes/u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 scale=1 1 1
- added link wrist_3_link, mass 0.18791; collision mesh filename=/home/iamnotedible/RR_Project/simulation/models/ur/meshes/u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 scale=1 1 1; visual mesh filename=/home/iamnotedible/RR_Project/simulation/models/ur/meshes/u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 scale=1 1 1
Joints:
- removed joint obstacle_joint
- added joint elbow_joint: type fixed, parent upper_arm_link, child forearm_link, origin xyz=0     -0.1197  0.425 rpy=0 0 0, axis 0 1 0, limit lower=-3.14159 upper=3.14159 effort=150.0 velocity=3.15
- added joint shoulder_lift_joint: type fixed, parent shoulder_link, child upper_arm_link, origin xyz=0      0.13585 0 rpy=3.14148 2.77079 3.14148, axis 0 1 0, limit lower=-6.28319 upper=6.28319 effort=150.0 velocity=3.15
- added joint shoulder_pan_joint: type fixed, parent UR_base_link, child shoulder_link, origin xyz=0      0      0.08915 rpy=0 0 -1.5708, axis 0 0 1, limit lower=-6.28319 upper=6.28319 effort=150.0 velocity=3.15
- added joint ur_pedestal_JOINT_1: type fixed, parent ur_pedestal, child UR_base_link, origin xyz=0 0 0 rpy=0 0 0, axis 0 0 0, limit lower=0 upper=0 effort=0 velocity=0
- added joint ur_pose: type fixed, parent world, child ur_pedestal, origin xyz=0.184218921 0.369103328 0.87 rpy=0.0 0.0 0.0622390961
- added joint wrist_1_joint: type fixed, parent forearm_link, child wrist_1_link, origin xyz=0      0      0.39225 rpy=0.39713 1.57078 0.39713, axis 0 1 0, limit lower=-6.28319 upper=6.28319 effort=28.0 velocity=3.2
- added joint wrist_2_joint: type fixed, parent wrist_1_link, child wrist_2_link, origin xyz=0    0.093 0 rpy=0 0 0, axis 0 0 1, limit lower=-6.28319 upper=6.28319 effort=28.0 velocity=3.2
- added joint wrist_3_joint: type fixed, parent wrist_2_link, child wrist_3_link, origin xyz=0      0      0.09465 rpy=0 0 0, axis 0 1 0, limit lower=-6.28319 upper=6.28319 effort=28.0 velocity=3.2
- joint sawyer_pose: origin xyz=0. 0. .9 rpy=0 0 0 -> xyz=0.25136679549411506 -0.5441101053518496 .78 rpy=0 0 1.60239812

Commit message: tes simplified

File: simulation/tes_planner/urdf/combined.urdf (robot description, URDF)
Before this commit: robot combined, 26 links, 25 joints
Links:
- link head: geometry collision sphere radius=0.18; visual mesh filename=/home/username/RR_Project/simulation/models/sawyer/meshes/s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
- link pedestal: geometry collision cylinder length=0.62 radius=0.18; visual mesh filename=/home/username/RR_Project/simulation/models/sawyer/meshes/s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
- link right_arm_base_link: geometry collision cylinder length=0.24 radius=0.08; visual mesh filename=/home/username/RR_Project/simulation/models/sawyer/meshes/s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
- link right_l0: geometry collision sphere radius=0.07; visual mesh filename=/home/username/RR_Project/simulation/models/sawyer/meshes/s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
- link right_l1: geometry collision sphere radius=0.07; visual mesh filename=/home/username/RR_Project/simulation/models/sawyer/meshes/s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
- link right_l2: geometry collision cylinder length=0.34 radius=0.06; visual mesh filename=/home/username/RR_Project/simulation/models/sawyer/meshes/s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
- link right_l3: geometry collision sphere radius=0.06; visual mesh filename=/home/username/RR_Project/simulation/models/sawyer/meshes/s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
- link right_l4: geometry collision cylinder length=0.30 radius=0.045; visual mesh filename=/home/username/RR_Project/simulation/models/sawyer/meshes/s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
- link right_l5: geometry collision sphere radius=0.06; visual mesh filename=/home/username/RR_Project/simulation/models/sawyer/meshes/s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
- link right_l6: geometry collision cylinder length=0.05 radius=0.055; visual mesh filename=/home/username/RR_Project/simulation/models/sawyer/meshes/s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
