Commit message: 1 iteration

File: urdf/combined.urdf (robot description, URDF)
Before this commit: robot combined, 35 links, 34 joints
Links:
- removed link b
- removed link base
- removed link base_link
- removed link ee_link
- removed link tool0
- added link ABB1200_base_link, mass 13.7742; collision mesh filename=model://abb/meshes/collision/base_link.stl scale=1 1 1; visual mesh filename=model://abb/meshes/visual/base_link.dae scale=1 1 1
- added link ABB1200_link_1, mass 11.8419; collision mesh filename=model://abb/meshes/collision/link_1.stl scale=1 1 1; visual mesh filename=model://abb/meshes/visual/link_1.dae scale=1 1 1
- added link ABB1200_link_2, mass 17.5394; collision mesh filename=model://abb/meshes/collision/link_2.stl scale=1 1 1; visual mesh filename=model://abb/meshes/visual/link_2.dae scale=1 1 1
- added link ABB1200_link_3, mass 7.46365; collision mesh filename=model://abb/meshes/collision/link_3.stl scale=1 1 1; visual mesh filename=model://abb/meshes/visual/link_3.dae scale=1 1 1
- added link ABB1200_link_4, mass 2.74436; collision mesh filename=model://abb/meshes/collision/link_4.stl scale=1 1 1; visual mesh filename=model://abb/meshes/visual/link_4.dae scale=1 1 1
- added link ABB1200_link_5, mass 0.62953; collision mesh filename=model://abb/meshes/collision/link_5.stl scale=1 1 1; visual mesh filename=model://abb/meshes/visual/link_5.dae scale=1 1 1
- added link ABB1200_link_6, mass 0.137; collision mesh filename=model://abb/meshes/collision/link_6.stl scale=1 1 1; visual mesh filename=model://abb/meshes/visual/link_6.dae scale=1 1 1
- added link UR_base_link, mass 4; collision mesh filename=model://ur/meshes/ur/collision/base.stl scale=1 1 1; visual mesh filename=model://ur/meshes/ur/visual/base.dae scale=1 1 1
- added link abb_pedestal, mass 1; visual cylinder length=1.0 radius=0.2
- added link sawyer_pedestal
- added link ur_pedestal, mass 1; visual cylinder length=1 radius=0.15
- link forearm_link: geometry collision mesh filename=model://ur/meshes/ur/collision/forearm.stl scale=1 1 1; visual mesh filename=model://ur/meshes/ur/visual/forearm.dae scale=1 1 1
- link head: geometry collision sphere radius=0.18; visual mesh filename=model://sawyer/meshes/sawyer_pv/head.DAE
- link pedestal: geometry visual mesh filename=model://sawyer/meshes/sawyer_pv/pedestal.DAE
- link right_arm_base_link: geometry collision cylinder length=0.24 radius=0.08; visual mesh filename=model://sawyer/meshes/sawyer_pv/base.DAE
- link right_l0: geometry collision sphere radius=0.07; visual mesh filename=model://sawyer/meshes/sawyer_mp3/l0.DAE
- link right_l1: geometry collision sphere radius=0.07; visual mesh filename=model://sawyer/meshes/sawyer_mp3/l1.DAE
- link right_l2: geometry collision cylinder length=0.34 radius=0.06; visual mesh filename=model://sawyer/meshes/sawyer_pv/l2.DAE
- link right_l3: geometry collision sphere radius=0.06; visual mesh filename=model://sawyer/meshes/sawyer_pv/l3.DAE
- link right_l4: geometry collision cylinder length=0.30 radius=0.045; visual mesh filename=model://sawyer/meshes/sawyer_pv/l4.DAE
- link right_l5: geometry collision sphere radius=0.06; visual mesh filename=model://sawyer/meshes/sawyer_pv/l5.DAE
- link right_l6: geometry collision cylinder length=0.05 radius=0.055; visual mesh filename=model://sawyer/meshes/sawyer_mp1/l6.DAE
- link shoulder_link: geometry collision mesh filename=model://ur/meshes/ur/collision/shoulder.stl scale=1 1 1; visual mesh filename=model://ur/meshes/ur/visual/shoulder.dae scale=1 1 1
- link upper_arm_link: geometry collision mesh filename=model://ur/meshes/ur/collision/upperarm.stl scale=1 1 1; visual mesh filename=model://ur/meshes/ur/visual/upperarm.dae scale=1 1 1
- link wrist_1_link: geometry collision mesh filename=model://ur/meshes/ur/collision/wrist1.stl scale=1 1 1; visual mesh filename=model://ur/meshes/ur/visual/wrist1.dae scale=1 1 1
- link wrist_2_link: geometry collision mesh filename=model://ur/meshes/ur/collision/wrist2.stl scale=1 1 1; visual mesh filename=model://ur/meshes/ur/visual/wrist2.dae scale=1 1 1
- link wrist_3_link: mass 0.1879 -> 0.18791; geometry collision mesh filename=model://ur/meshes/ur/collision/wrist3.stl scale=1 1 1; visual mesh filename=model://ur/meshes/ur/visual/wrist3.dae scale=1 1 1
Joints:
- removed joint b_link-base_fixed_joint
- removed joint base_link-base_fixed_joint
- removed joint ee_fixed_joint
- removed joint world_joint
- removed joint wrist_3_link-tool0_fixed_joint
- added joint ABB1200_joint_1: type revolute, parent ABB1200_base_link, child ABB1200_link_1, origin xyz=0     0     0.3991 rpy=0 0 0, axis 0 0 1, limit lower=-2.967 upper=2.967 effort=1000.0 velocity=5.027
- added joint ABB1200_joint_2: type revolute, parent ABB1200_link_1, child ABB1200_link_2, origin xyz=0 0 0 rpy=0 0 0, axis 0 1 0, limit lower=-1.745 upper=2.269 effort=1000.0 velocity=4.189
- added joint ABB1200_joint_3: type revolute, parent ABB1200_link_2, child ABB1200_link_3, origin xyz=0    0    0.448 rpy=0 0 0, axis 0 1 0, limit lower=-3.491 upper=1.222 effort=1000.0 velocity=5.236
- added joint ABB1200_joint_4: type revolute, parent ABB1200_link_3, child ABB1200_link_4, origin xyz=0    0    0.042 rpy=0 0 0, axis 1 0 0, limit lower=-4.712 upper=4.712 effort=1000.0 velocity=6.981
- added joint ABB1200_joint_5: type revolute, parent ABB1200_link_4, child ABB1200_link_5, origin xyz=0.451 0    0 rpy=0 0 0, axis 0 1 0, limit lower=-2.269 upper=2.269 effort=1000.0 velocity=7.069
- added joint ABB1200_joint_6: type revolute, parent ABB1200_link_5, child ABB1200_link_6, origin xyz=0.082 0    0 rpy=0 0 0, axis 1 0 0, limit lower=-6.283 upper=6.283 effort=1000.0 velocity=10.472
- added joint abb_pedestal_JOINT_0: type fixed, parent abb_pedestal, child ABB1200_base_link, origin xyz=0 0 0 rpy=0 0 0, axis 0 0 0, limit lower=0 upper=0 effort=0 velocity=0
- added joint abb_pose: type fixed, parent world, child abb_pedestal, origin xyz=0 1.2 0.0 rpy=0.0 0.0 0.0
- added joint sawyer_pose: type fixed, parent world, child sawyer_pedestal, origin xyz=0. 0. 0.11 rpy=0 0 0
- added joint ur_pedestal_JOINT_1: type fixed, parent ur_pedestal, child UR_base_link, origin xyz=0 0 0 rpy=0 0 0, axis 0 0 0, limit lower=0 upper=0 effort=0 velocity=0
- added joint ur_pose: type fixed, parent world, child ur_pedestal, origin xyz=1.2 0 0.0 rpy=0.0 0.0 1.57
- joint controller_box_fixed: parent b -> sawyer_pedestal
- joint elbow_joint: limit lower=-3.14159265359 upper=3.14159265359 effort=150.0 velocity=3.15 -> lower=-3.14159 upper=3.14159 effort=150.0 velocity=3.15; origin xyz=0.0 -0.1197 0.425 rpy=0.0 0.0 0.0 -> xyz=0     -0.1197  0.425 rpy=0 0 0
- joint pedestal_feet_fixed: parent b -> sawyer_pedestal
- joint pedestal_fixed: parent b -> sawyer_pedestal
- joint right_arm_mount: parent b -> sawyer_pedestal
- joint shoulder_lift_joint: limit lower=-6.28318530718 upper=6.28318530718 effort=150.0 velocity=3.15 -> lower=-6.28319 upper=6.28319 effort=150.0 velocity=3.15; origin xyz=0.0 0.13585 0.0 rpy=0.0 1.57079632679 0.0 -> xyz=0      0.13585 0 rpy=3.14148 1.57079 3.14148
- joint shoulder_pan_joint: limit lower=-6.28318530718 upper=6.28318530718 effort=150.0 velocity=3.15 -> lower=-6.28319 upper=6.28319 effort=150.0 velocity=3.15; origin xyz=0.0 0.0 0.089159 rpy=0.0 0.0 0.0 -> xyz=0      0      0.08915 rpy=0 0 0; parent base_link -> UR_base_link
- joint torso_t0: parent b -> sawyer_pedestal
- joint wrist_1_joint: limit lower=-6.28318530718 upper=6.28318530718 effort=28.0 velocity=3.2 -> lower=-6.28319 upper=6.28319 effort=28.0 velocity=3.2; origin xyz=0.0 0.0 0.39225 rpy=0.0 1.57079632679 0.0 -> xyz=0      0      0.39225 rpy=0.39713 1.57078 0.39713
- joint wrist_2_joint: limit lower=-6.28318530718 upper=6.28318530718 effort=28.0 velocity=3.2 -> lower=-6.28319 upper=6.28319 effort=28.0 velocity=3.2; origin xyz=0.0 0.093 0.0 rpy=0.0 0.0 0.0 -> xyz=0    0.093 0 rpy=0 0 0
- joint wrist_3_joint: limit lower=-6.28318530718 upper=6.28318530718 effort=28.0 velocity=3.2 -> lower=-6.28319 upper=6.28319 effort=28.0 velocity=3.2; origin xyz=0.0 0.0 0.09465 rpy=0.0 0.0 0.0 -> xyz=0      0      0.09465 rpy=0 0 0

File: urdf/sawyer.urdf (robot description, URDF)
Before this commit: robot sawyer, 24 links, 23 joints
Links:
- link head: geometry collision sphere radius=0.18; visual mesh filename=package://sawyer_description/meshes/sawyer_pv/head.DAE
- link pedestal: geometry collision cylinder length=0.62 radius=0.18; visual mesh filename=package://sawyer_description/meshes/sawyer_pv/pedestal.DAE
- link right_arm_base_link: geometry collision cylinder length=0.24 radius=0.08; visual mesh filename=package://sawyer_description/meshes/sawyer_pv/base.DAE
- link right_l0: geometry collision sphere radius=0.07; visual mesh filename=package://sawyer_description/meshes/sawyer_mp3/l0.DAE
- link right_l1: geometry collision sphere radius=0.07; visual mesh filename=package://sawyer_description/meshes/sawyer_mp3/l1.DAE
- link right_l2: geometry collision cylinder length=0.34 radius=0.06; visual mesh filename=package://sawyer_description/meshes/sawyer_pv/l2.DAE
- link right_l3: geometry collision sphere radius=0.06; visual mesh filename=package://sawyer_description/meshes/sawyer_pv/l3.DAE
- link right_l4: geometry collision cylinder length=0.30 radius=0.045; visual mesh filename=package://sawyer_description/meshes/sawyer_pv/l4.DAE
- link right_l5: geometry collision sphere radius=0.06; visual mesh filename=package://sawyer_description/meshes/sawyer_pv/l5.DAE
- link right_l6: geometry collision cylinder length=0.05 radius=0.055; visual mesh filename=package://sawyer_description/meshes/sawyer_mp1/l6.DAE

Commit message: urdf with gripper box

File: urdf/combined.urdf (robot description, URDF)
Before this commit: robot combined, 41 links, 40 joints
Links:
- added link ABB1200_link_7, mass 0.137; collision box size=0.03 0.08 0.08; visual box size=0.08 0.08 0.03
- added link UR_link_7, mass 0.137; collision box size=0.03 0.08 0.08; visual box size=0.08 0.08 0.03
Joints:
- added joint UR_gripper_joint: type fixed, parent wrist_3_link, child UR_link_7, origin xyz=0 0 0 rpy=0 0 0, axis 0 0 0, limit lower=0 upper=0 effort=0 velocity=0
- added joint link_6_JOINT_0: type fixed, parent ABB1200_link_6, child ABB1200_link_7, origin xyz=0 0 0 rpy=0 0 0, axis 0 0 0, limit lower=0 upper=0 effort=0 velocity=0
